File: Kugelilift.kicad_pcb (KiCad board)
At the start: 2 copper layers, 43 x 43.5 mm, 13 parts, among them J2 TTL, J4 Stepper, SW1 RESET, SW2 MODE, U1 magnetic-charger, U2 TCRT5000, U3 ULN2003A, U5 UA78M33_TO252, U6 esp-01m

Commit message: Small rearrangements
Parts:
- moved SW1 2.78 mm to (103.6, 77.6)
Routing:
- net Net-(SW1-Pad1): track 6.32 -> 3.37 mm
- net Net-(R1-Pad2): track 23.5 -> 24.7 mm
- net unconnected-(U6-Pad11): track 6.38 -> 5.81 mm
Changed lines of the file:
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@@
   )
   (footprint "Connector_PinHeader_2.54mm:PinHeader_1x03_P2.54mm_Vertical" (layer "F.Cu")
-    (at 104.236652 80.292439)
+    (at 103.627074 77.582928)
     (descr "Through hole straight pin header, 1x03, 2.54mm pitch, single row")
     (tags "Through hole pin header THT 1x03 2.54mm single row")
@@
   (segment (start 115.6 96.737612) (end 115.770559 96.908171) (width 0.46) (layer "B.Cu") (net 2))
   (segment (start 141.155 78.075) (end 140.28 77.2) (width 0.8) (layer "B.Cu") (net 2))
-  (segment (start 107.98 80.898574) (end 110 78.878574) (width 0.46) (layer "B.Cu") (net 8))
-  (segment (start 110 78.878574) (end 110 74.219243) (width 0.46) (layer "B.Cu") (net 8))
-  (segment (start 107.98 85.09495) (end 107.98 80.898574) (width 0.46) (layer "B.Cu") (net 8))
-  (segment (start 108.479988 75.067488) (end 108.479988 78.617382) (width 0.46) (layer "B.Cu") (net 9))
-  (segment (start 106.720499 80.376871) (end 106.720499 81.731444) (width 0.46) (layer "B.Cu") (net 9))
-  (segment (start 108.479988 78.617382) (end 106.720499 80.376871) (width 0.46) (layer "B.Cu") (net 9))
-  (segment (start 106.71 81.741943) (end 106.71 85.75) (width 0.46) (layer "B.Cu") (net 9))
-  (segment (start 108.4125 75) (end 108.479988 75.067488) (width 0.46) (layer "B.Cu") (net 9))
-  (segment (start 106.720499 81.731444) (end 106.71 81.741943) (width 0.46) (layer "B.Cu") (net 9))
-  (segment (start 111.5875 79.072277) (end 109.25 81.409777) (width 0.46) (layer "B.Cu") (net 10))
-  (segment (start 111.5875 75) (end 111.5875 79.072277) (width 0.46) (layer "B.Cu") (net 10))
-  (segment (start 109.25 81.409777) (end 109.25 85.75) (width 0.46) (layer "B.Cu") (net 10))
+  (segment (start 107.98 82.069026) (end 110 80.049026) (width 0.46) (layer "B.Cu") (net 8))
+  (segment (start 110 80.049026) (end 110 74.219243) (width 0.46) (layer "B.Cu") (net 8))
+  (segment (start 107.98 85.09495) (end 107.98 82.069026) (width 0.46) (layer "B.Cu") (net 8))
+  (segment (start 108.4125 79.855323) (end 106.71 81.557823) (width 0.46) (layer "B.Cu") (net 9))
+  (segment (start 106.71 81.557823) (end 106.71 85.75) (width 0.46) (layer "B.Cu") (net 9))
+  (segment (start 108.4125 75) (end 108.4125 79.855323) (width 0.46) (layer "B.Cu") (net 9))
+  (segment (start 109.25 82.58023) (end 109.25 85.75) (width 0.46) (layer "B.Cu") (net 10))
+  (segment (start 111.449032 80.381198) (end 109.25 82.58023) (width 0.46) (layer "B.Cu") (net 10))
+  (segment (start 111.5875 75) (end 111.449032 75.138468) (width 0.46) (layer "B.Cu") (net 10))
+  (segment (start 111.449032 75.138468) (end 111.449032 80.381198) (width 0.46) (layer "B.Cu") (net 10))
   (segment (start 120.730002 80.749998) (end 120.730002 84.049998) (width 0.46) (layer "B.Cu") (net 12))
   (segment (start 120.730002 84.049998) (end 120.38 84.4) (width 0.46) (layer "B.Cu") (net 12))
@@
   (segment (start 106.825 70.269243) (end 106.825 68.309243) (width 0.46) (layer "B.Cu") (net 14))
   (segment (start 108.662594 66.471649) (end 112.297837 66.471649) (width 0.46) (layer "B.Cu") (net 14))
-  (segment (start 106.133768 77.32988) (end 117.034309 77.32988) (width 0.46) (layer "F.Cu") (net 19))
-  (segment (start 117.034309 77.32988) (end 117.176719 77.47229) (width 0.46) (layer "F.Cu") (net 19))
-  (segment (start 105.757922 77.705726) (end 106.133768 77.32988) (width 0.46) (layer "F.Cu") (net 19))
-  (via (at 105.757922 77.705726) (size 2) (drill 1) (layers "F.Cu" "B.Cu") (net 19))
+  (segment (start 107.925386 77.47229) (end 106.259581 79.138095) (width 0.46) (layer "F.Cu") (net 19))
+  (segment (start 117.176719 77.47229) (end 107.925386 77.47229) (width 0.46) (layer "F.Cu") (net 19))
+  (via (at 106.259581 79.138095) (size 2) (drill 1) (layers "F.Cu" "B.Cu") (net 19))
   (via (at 117.176719 77.47229) (size 2) (drill 1) (layers "F.Cu" "B.Cu") (net 19))
+  (segment (start 106.825 75) (end 106.825 78.572676) (width 0.46) (layer "B.Cu") (net 19))
   (segment (start 121.84 74.14) (end 121.84 71.878405) (width 0.46) (layer "B.Cu") (net 19))
   (segment (start 117.176719 76.813281) (end 117.176719 77.47229) (width 0.46) (layer "B.Cu") (net 19))
-  (segment (start 106.825 75) (end 106.825 76.638648) (width 0.46) (layer "B.Cu") (net 19))
   (segment (start 118.740002 75.249998) (end 117.176719 76.813281) (width 0.46) (layer "B.Cu") (net 19))
-  (segment (start 106.825 76.638648) (end 105.757922 77.705726) (width 0.46) (layer "B.Cu") (net 19))
+  (segment (start 106.825 78.572676) (end 106.259581 79.138095) (width 0.46) (layer "B.Cu") (net 19))
   (segment (start 120.730002 75.249998) (end 121.84 74.14) (width 0.46) (layer "B.Cu") (net 19))
   (segment (start 120.730002 75.249998) (end 118.740002 75.249998) (width 0.46) (layer "B.Cu") (net 19))
-  (segment (start 104.236652 80.292439) (end 103.65 79.705787) (width 0.46) (layer "B.Cu") (net 20))
-  (segment (start 103.65 79.705787) (end 103.65 74.219243) (width 0.46) (layer "B.Cu") (net 20))
+  (segment (start 103.65 77.560002) (end 103.65 74.219243) (width 0.46) (layer "B.Cu") (net 20))
+  (segment (start 103.627074 77.582928) (end 103.65 77.560002) (width 0.46) (layer "B.Cu") (net 20))
   (segment (start 118.537802 68.535291) (end 118.706025 68.703514) (width 0.46) (layer "F.Cu") (net 21))
   (segment (start 122.094869 68.703514) (end 122.827883 67.9705) (width 0.46) (layer "F.Cu") (net 21))
@@
   (segment (start 114.7625 68.066743) (end 115.09 67.739243) (width 0.46) (layer "B.Cu") (net 21))
   (segment (start 114.7625 70) (end 114.7625 68.066743) (width 0.46) (layer "B.Cu") (net 21))
-  (segment (start 110.52 85.75) (end 110.52 81.92098) (width 0.46) (layer "B.Cu") (net 22))
-  (segment (start 110.52 81.92098) (end 113.075695 79.365285) (width 0.46) (layer "B.Cu") (net 22))
-  (segment (start 113.075695 75.099305) (end 113.175 75) (width 0.46) (layer "B.Cu") (net 22))
-  (segment (start 113.075695 79.365285) (end 113.075695 75.099305) (width 0.46) (layer "B.Cu") (net 22))
+  (segment (start 110.52 83.09214) (end 113.175 80.43714) (width 0.46) (layer "B.Cu") (net 22))
+  (segment (start 110.52 85.75) (end 110.52 83.09214) (width 0.46) (layer "B.Cu") (net 22))
+  (segment (start 113.175 80.43714) (end 113.175 75) (width 0.46) (layer "B.Cu") (net 22))
   (segment (start 110.52 92.25) (end 110.52 97.018113) (width 0.46) (layer "B.Cu") (net 23))
   (segment (start 110.52 97.018113) (end 110.498524 97.039589) (width 0.46) (layer "B.Cu") (net 23))
@@
   (segment (start 106.71 92.25) (end 106.71 93.202234) (width 0.46) (layer "B.Cu") (net 26))
   (segment (start 102.998524 96.91371) (end 102.998524 97.039589) (width 0.46) (layer "B.Cu") (net 26))
-  (via (at 114.777286 80.596498) (size 2) (drill 1) (layers "F.Cu" "B.Cu") (net 29))
-  (segment (start 114.7625 74.219243) (end 114.7625 80.581712) (width 0.46) (layer "B.Cu") (net 29))
-  (segment (start 114.7625 80.581712) (end 114.777286 80.596498) (width 0.46) (layer "B.Cu") (net 29))
+  (via (at 115.477814 79.737608) (size 2) (drill 1) (layers "F.Cu" "B.Cu") (net 29))
+  (segment (start 114.7625 74.219243) (end 114.7625 79.022294) (width 0.46) (layer "B.Cu") (net 29))
+  (segment (start 114.7625 79.022294) (end 115.477814 79.737608) (width 0.46) (layer "B.Cu") (net 29))
   (zone (net 3) (net_name "GND") (layer "B.Cu") (hatch edge 0.508)
     (connect_pads (clearance 0.508))

Commit message: Final adjustments
Parts:
- moved C2 19.8 mm to (129.1, 79.4), turned to 0 degrees
- moved U1 12.5 mm to (134.3, 90.1), turned to 135 degrees
- moved J4 5.62 mm to (118.6, 97.3)
- moved C1 5.38 mm to (140.0, 81.6), turned to 180 degrees
- moved U3 2.34 mm to (113.3, 87.4)
- moved U5 1.00 mm to (137.0, 73.0)
- moved J2 0.38 mm to (111.0, 64.6)
- moved SW1 0.22 mm to (103.8, 77.4)
Routing:
- net +3V3: track 77.4 -> 60.5 mm
- net +5V: track 47.0 -> 42.5 mm
- net Net-(J4-Pad2): track 4.80 -> 8.13 mm
- net Net-(R1-Pad2): track 24.7 -> 22.0 mm
- net /in-4: track 11.8 -> 9.44 mm
- net Net-(J4-Pad3): track 5.31 -> 7.60 mm
- net /in-3: track 11.7 -> 9.52 mm
- net /in-1: track 11.5 -> 9.30 mm
- net /in-2: track 11.7 -> 9.94 mm
- net Net-(J4-Pad4): track 5.82 -> 7.19 mm
Other:
- outline, holes or cut-outs redrawn
- board text added: "Kugelilift v2.3 17.12.23"
- board text removed: "Kugelilift v2.3 16.12.23"

Commit message: Prepare for milling
Connections:
- U6 pad 7: unconnected-(U6-Pad7) -> +3V3
Other:
- board text added: "Kugelilift v2.3 21.12.23"
- board text removed: "Kugelilift v2.3 17.12.23"

Commit message: Prepare for next iteration
Parts:
- added SW3: SW_Push, Button_Switch_SMD:SW_Push_1P1T_NO_CK_KMR2, F.Cu at (109.2, 111.8)
- added SW4: SW_DIP_x04, Button_Switch_THT:SW_DIP_SPSTx04_Slide_6.7x11.72mm_W7.62mm_P2.54mm_LowProfile, F.Cu at (117.2, 108.0)
- added SW5: SW_Push, Button_Switch_SMD:SW_Push_1P1T_NO_CK_KMR2, F.Cu at (98.8, 111.8)
Connections:
- U6 pad 7: +3V3 -> unconnected-(U6-Pad7)
Other:
- board text added: "23.01.2024"
- board text added: "Kugelilift v3.0-beta"
- board text removed: "Kugelilift v2.3 21.12.23"
